File: tracker/hardware/output/v2_adc_freerouted.kicad_pcb (KiCad board)
At the start: 2 copper layers, 50 x 40 mm, 17 parts, among them U1 ESP32-C3, U2 LR2021F33, U3 MAX-M10S, U4 TPS7A02

Commit message: fix: ESP32-C3 GPIO5/GPIO6 pad collision — shift bottom row inboard by one pitch
Routing:
- net SPI_MISO: track 23.2 -> 18.5 mm
- net VDIV_MID: track 3.00 -> 0.00 mm
- net GND: track 148.4 -> 145.6 mm
Changed lines of the file:
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@@
 		)
 		(pad "GPIO5" smd rect
-			(at -3.5 4.25)
-			(size 0.6 0.4)
+			(at -3.5 3.75)
+			(size 1 0.6)
 			(layers "F.Cu" "F.Mask")
 			(net 9 "LR2021_DIO9")
@@
 		(pad "GPIO6" smd rect
 			(at -3 3.5)
-			(size 0.8 0.5)
+			(size 1 0.6)
 			(layers "F.Cu" "F.Mask")
 			(net 3 "SPI_SCK")
@@
 		(pad "GPIO7" smd rect
 			(at -1.5 3.5)
-			(size 0.8 0.5)
+			(size 1 0.6)
 			(layers "F.Cu" "F.Mask")
 			(net 4 "SPI_MOSI")
@@
 		(pad "GPIO9" smd rect
 			(at 1.5 3.5)
-			(size 0.8 0.5)
+			(size 1 0.6)
 			(layers "F.Cu" "F.Mask")
 			(net 11 "STATUS_LED")
@@
 		(pad "GPIO10" smd rect
 			(at 3 3.5)
-			(size 0.8 0.5)
+			(size 1 0.6)
 			(layers "F.Cu" "F.Mask")
 			(net 6 "SPI_NSS")
@@
 	)
 	(segment
-		(start 3.5 32)
-		(end 5.3 32)
-		(width 0.2)
-		(layer "F.Cu")
-		(net 2)
-	)
-	(segment
 		(start 34.9 31)
 		(end 34.9 29)
@@
 		(end 34.5517 37)
 		(width 2)
-		(layer "F.Cu")
-		(net 2)
-	)
-	(segment
-		(start 5.3 32)
-		(end 5.3 33)
-		(width 0.2)
 		(layer "F.Cu")
 		(net 2)
@@
 	)
 	(segment
-		(start 10.5 14)
-		(end 10.5 11.25)
-		(width 0.2)
-		(layer "B.Cu")
-		(net 5)
-	)
-	(segment
-		(start 10.5 11.25)
-		(end 8.5 11.25)
-		(width 0.2)
-		(layer "B.Cu")
-		(net 5)
-	)
-	(segment
 		(start 13.6315 20.9496)
 		(end 16.2134 20.9496)
@@
 		(net 17)
 	)
-	(segment
-		(start 3.5 31.4)
-		(end 3.5 30)
-		(width 0.2)
-		(layer "F.Cu")
-		(net 18)
-	)
-	(segment
-		(start 2.5 31.4)
-		(end 3.5 31.4)
-		(width 0.2)
-		(layer "F.Cu")
-		(net 18)
-	)
-	(segment
-		(start 2.5 32)
-		(end 2.5 31.4)
-		(width 0.2)
-		(layer "F.Cu")
-		(net 18)
-	)
 	(embedded_fonts no)
