File: tracker/hardware/output/v8j_u5net.kicad_pcb (KiCad board)
At the start: 4 copper layers, 55 x 45 mm, 28 parts, among them J1 Prog_Header, J2 Debug_Header, U1 ESP32-C3-WROOM-02, U2 LoRa2021_Gen4, U3 MAX-M10S, U4 TPS7A02, U5 MS5611-01BA

Commit message: fix(hw): v8j U5 MS5611 nets + zone refill -> 0 unconnected, 159/159 DRC errors cleared (5 under-size vias left)
Routing:
- net GND: track 119.1 -> 100.9 mm, vias 15 -> 14
- net EN: track 48.8 -> 30.6 mm
- net I2C_SCL: track 61.2 -> 43.8 mm, vias 5 -> 2
- net I2C_SDA: track 60.8 -> 43.5 mm, vias 3 -> 2
- net +3V3: track 68.0 -> 54.8 mm, vias 10 -> 8
