File: tracker/hardware/wing_board/wing_board_v9.kicad_pcb (KiCad board)
At the start: 2 copper layers, 184 x 25 mm, 12 parts, among them J1 WingTab_v9_4pin

Commit message: feat(hw/wing): parametric 3D models for the v9 wing — the 3 cells now render
The v9 wing board carried no 3D model on ANY of its 12 placed references, so a
render showed a bare FR4 outline: the three solar cells the wing exists to fly
were invisible. The hub board's models are worse than absent -- they point at
${KICAD9_3DMODEL_DIR}/...step, i.e. at kicad-packages3d (4.77 GB, NOT installed
here and not installable: ~2.3 GB free).

Added, all plain text and committed, so a render resolves with nothing installed:
  * scripts/gen_3d_models_wing.py  -- parametric VRML generator, `--check` mode
    fails closed on a stale tree. Its docstring carries the MEASURED KiCad model
    convention: 1 VRML unit = 2.54 mm, X = footprint +x, Y = -(footprint +y),
    Z = up with Z=0 at the board top face. Measured twice (a throwaway probe board
    round-tripped through `kicad-cli pcb export vrml --units mm`, plus the shipped
    ecc83.wrl demo model: 8.86 units = 22.5 mm envelope vs a 21.2 mm courtyard).
  * tracker/hardware/3dmodels/cells/  -- the SMALL cell 52.07 x 19.65 x 0.21
    (ADR-049 measured inputs; the board's own footprint is SolarCell_52x19mm) as
    the wing's cell model, plus the LARGE 78.55 x 38.90 x 0.21 as a SHARED,
    unassigned asset for the hub/array direction. cells/ is named for sharing so
    the parallel hub worker reuses them instead of duplicating.
  * tracker/hardware/3dmodels/wing/   -- J1's four 4.0x1.2 lands at 1.8 mm pitch,
    the FID1-3 1 mm dots, the FB1 0402 body (DNP -> rendered translucent so it
    cannot be mistaken for a fitted part), and RF1's V2 provision land.
  * build_wing_v9.py + the regenerated board: +99 lines / 0 deletions, all of it
    (model ...) metadata. Proven unchanged by parsing both revisions and
    set-comparing nets (17), footprints (12 with lib id / ref / position / every
    pad), segments (8), Edge.Cuts (8), gr_text (1) and thickness. No net, no part
    position and no ADR decision was touched. Two generator runs are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
Parts:
- removed the FB1 at (58.0, 1.70)
- removed the FID3 at (145.0, 1.70)
- removed the H1 at (8.00, 1.70)
- added FID1: Fiducial_1mm_Mask2mm, WingV9:Fiducial_1mm_Mask2mm, F.Cu at (30.0, 1.70)
- added FID2: Fiducial_1mm_Mask2mm, WingV9:Fiducial_1mm_Mask2mm, F.Cu at (105.0, 1.70)
- added J1: WingTab_v9_4pin, WingV9:WingTab_v9_4pin, F.Cu at (0.00, 0.00)
- FB1: renamed from FID2; value Fiducial_1mm_Mask2mm -> FerriteBead_0402_DNP_V2only; footprint WingV9:Fiducial_1mm_Mask2mm -> WingV9:FerriteBead_0402_V2provision
- H1: renamed from J1; value WingTab_v9_4pin -> MountingHole_NPTH_2.2mm; footprint WingV9:WingTab_v9_4pin -> WingV9:MountingHole_2.2mm_NPTH
- moved FID3 115.0 mm to (145.0, 1.70)
- moved FB1 47.0 mm to (58.0, 1.70)
- moved H1 8.18 mm to (8.00, 1.70)
- renumbered FID1 to FID3
Changed lines of the file:
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@@
     (pad "1" smd rect (at -28 0) (size 1.6 4) (layers "F.Cu" "F.Paste" "F.Mask") (net 1 "SOLAR_P"))
     (pad "2" smd rect (at 28 0) (size 1.6 4) (layers "F.Cu" "F.Paste" "F.Mask") (net 3 "SOLAR_MID1"))
-    (fp_rect (start -29.05 -9.75) (end 29.05 9.75)
-     (stroke (width 0.05) (type solid)) (fill no) (layer "F.CrtYd"))
+    (model "${KIPRJMOD}/../3dmodels/cells/solar_cell_small_52.07x19.65x0.21.wrl"
+      (offset
+        (xyz 0 0 0)
+      )
+      (scale
+        (xyz 1 1 1)
+      )
+      (rotate
+        (xyz 0 0 0)
+      )
+    )
   )
   (footprint "WingV9:SolarCell_52x19mm"
@@
     (pad "1" smd rect (at -28 0) (size 1.6 4) (layers "F.Cu" "F.Paste" "F.Mask") (net 3 "SOLAR_MID1"))
     (pad "2" smd rect (at 28 0) (size 1.6 4) (layers "F.Cu" "F.Paste" "F.Mask") (net 4 "SOLAR_MID2"))
-    (fp_rect (start -29.05 -9.75) (end 29.05 9.75)
-     (stroke (width 0.05) (type solid)) (fill no) (layer "F.CrtYd"))
+    (model "${KIPRJMOD}/../3dmodels/cells/solar_cell_small_52.07x19.65x0.21.wrl"
+      (offset
+        (xyz 0 0 0)
+      )
+      (scale
+        (xyz 1 1 1)
+      )
+      (rotate
+        (xyz 0 0 0)
+      )
+    )
   )
   (footprint "WingV9:SolarCell_52x19mm"
@@
     (pad "1" smd rect (at -28 0) (size 1.6 4) (layers "F.Cu" "F.Paste" "F.Mask") (net 4 "SOLAR_MID2"))
     (pad "2" smd rect (at 28 0) (size 1.6 4) (layers "F.Cu" "F.Paste" "F.Mask") (net 2 "SOLAR_N"))
-    (fp_rect (start -29.05 -9.75) (end 29.05 9.75)
-     (stroke (width 0.05) (type solid)) (fill no) (layer "F.CrtYd"))
+    (model "${KIPRJMOD}/../3dmodels/cells/solar_cell_small_52.07x19.65x0.21.wrl"
+      (offset
+        (xyz 0 0 0)
+      )
+      (scale
+        (xyz 1 1 1)
+      )
+      (rotate
+        (xyz 0 0 0)
+      )
+    )
   )
   (footprint "WingV9:WingTab_v9_4pin"
@@
     (fp_text user "N" (at -5 16.9) (layer "F.SilkS") (effects (font (size 0.6 0.6) (thickness 0.1))))
     (fp_rect (start -7 8.4) (end -3 16.6) (stroke (width 0.1) (type solid)) (fill none) (layer "F.SilkS"))
-    (fp_rect (start -7.25 8.95) (end -2.75 16.05)
-     (stroke (width 0.05) (type solid)) (fill no) (layer "F.CrtYd"))
+    (model "${KIPRJMOD}/../3dmodels/wing/wing_v9_tab_4pin_lands.wrl"
+      (offset
+        (xyz 0 0 0)
+      )
+      (scale
+        (xyz 1 1 1)
+      )
+      (rotate
+        (xyz 0 0 0)
+      )
+    )
   )
   (footprint "WingV9:MountingHole_2.2mm_NPTH"
@@
     )
     (pad "" np_thru_hole circle (at 0 0) (size 2.2 2.2) (drill 2.2) (layers "*.Cu" "*.Mask"))
-    (fp_circle (center 0 0) (end 1.35 0)
-     (stroke (width 0.05) (type solid)) (fill no) (layer "F.CrtYd"))
   )
   (footprint "WingV9:MountingHole_2.2mm_NPTH"
@@
     )
     (pad "" np_thru_hole circle (at 0 0) (size 2.2 2.2) (drill 2.2) (layers "*.Cu" "*.Mask"))
-    (fp_circle (center 0 0) (end 1.35 0)
-     (stroke (width 0.05) (type solid)) (fill no) (layer "F.CrtYd"))
   )
   (footprint "WingV9:MountingHole_2.2mm_NPTH"
@@
     )
     (pad "" np_thru_hole circle (at 0 0) (size 2.2 2.2) (drill 2.2) (layers "*.Cu" "*.Mask"))
-    (fp_circle (center 0 0) (end 1.35 0)
-     (stroke (width 0.05) (type solid)) (fill no) (layer "F.CrtYd"))
   )
   (footprint "WingV9:Fiducial_1mm_Mask2mm"
@@
     (attr smd)
     (pad "1" smd circle (at 0 0) (size 1 1) (layers "F.Cu" "F.Mask"))
-    (fp_circle (center 0 0) (end 1.25 0)
-     (stroke (width 0.05) (type solid)) (fill no) (layer "F.CrtYd"))
+    (model "${KIPRJMOD}/../3dmodels/wing/wing_v9_fiducial_1mm_dot.wrl"
+      (offset
+        (xyz 0 0 0)
+      )
+      (scale
+        (xyz 1 1 1)
+      )
+      (rotate
+        (xyz 0 0 0)
+      )
+    )
   )
   (footprint "WingV9:Fiducial_1mm_Mask2mm"
@@
     (attr smd)
     (pad "1" smd circle (at 0 0) (size 1 1) (layers "F.Cu" "F.Mask"))
-    (fp_circle (center 0 0) (end 1.25 0)
-     (stroke (width 0.05) (type solid)) (fill no) (layer "F.CrtYd"))
+    (model "${KIPRJMOD}/../3dmodels/wing/wing_v9_fiducial_1mm_dot.wrl"
+      (offset
+        (xyz 0 0 0)
+      )
+      (scale
+        (xyz 1 1 1)
+      )
+      (rotate
+        (xyz 0 0 0)
+      )
+    )
   )
   (footprint "WingV9:Fiducial_1mm_Mask2mm"
@@
     (attr smd)
     (pad "1" smd circle (at 0 0) (size 1 1) (layers "F.Cu" "F.Mask"))
-    (fp_circle (center 0 0) (end 1.25 0)
-     (stroke (width 0.05) (type solid)) (fill no) (layer "F.CrtYd"))
+    (model "${KIPRJMOD}/../3dmodels/wing/wing_v9_fiducial_1mm_dot.wrl"
+      (offset
+        (xyz 0 0 0)
+      )
+      (scale
+        (xyz 1 1 1)
+      )
+      (rotate
+        (xyz 0 0 0)
+      )
+    )
   )
   (footprint "WingV9:FerriteBead_0402_V2provision"
@@
     (pad "1" smd rect (at -0.45 0) (size 0.5 0.6) (layers "F.Cu" "F.Paste" "F.Mask"))
     (pad "2" smd rect (at 0.45 0) (size 0.5 0.6) (layers "F.Cu" "F.Paste" "F.Mask"))
-    (fp_rect (start -0.95 -0.55) (end 0.95 0.55)
-     (stroke (width 0.05) (type solid)) (fill no) (layer "F.CrtYd"))
+    (model "${KIPRJMOD}/../3dmodels/wing/ferrite_bead_0402_dnp.wrl"
+      (offset
+        (xyz 0 0 0)
+      )
+      (scale
+        (xyz 1 1 1)
+      )
+      (rotate
+        (xyz 0 0 0)
+      )
+    )
   )
   (footprint "WingV9:RF_ProvisionPad_v2only"
@@
     (attr smd)
     (pad "1" smd rect (at 0 0) (size 2 2) (layers "F.Cu" "F.Mask"))
-    (fp_rect (start -1.25 -1.25) (end 1.25 1.25)
-     (stroke (width 0.05) (type solid)) (fill no) (layer "F.CrtYd"))
+    (model "${KIPRJMOD}/../3dmodels/wing/wing_v9_rf_provision_pad_2x2.wrl"
+      (offset
+        (xyz 0 0 0)
+      )
+      (scale
+        (xyz 1 1 1)
+      )
+      (rotate
+        (xyz 0 0 0)
+      )
+    )
   )
   (segment (start 2 12.5) (end 2 9.8)

Commit message: feat(wing): add ADR-065 double-sided solar cells
Parts:
- added FID2: Fiducial_1mm_Mask2mm, WingV9:Fiducial_1mm_Mask2mm, F.Cu at (105.0, 1.70)
- added SC4: SolarCell_52x19mm_0.5V, WingV9:SolarCell_52x19mm, B.Cu at (30.0, 12.5)
- added SC5: SolarCell_52x19mm_0.5V, WingV9:SolarCell_52x19mm, B.Cu at (88.0, 12.5)
- SC6: renamed from FID2; value Fiducial_1mm_Mask2mm -> SolarCell_52x19mm_0.5V; footprint WingV9:Fiducial_1mm_Mask2mm -> WingV9:SolarCell_52x19mm; moved to B.Cu
- moved SC6 42.4 mm to (146.0, 12.5)
Connections:
- SC6 pad 1: (no net) -> SOLAR_MID2
Changed lines of the file:
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@@
     (fp_text user "+" (at -26 23.6) (layer "F.SilkS") (effects (font (size 1 1) (thickness 0.12))))
     (fp_text user "-" (at 26 23.6) (layer "F.SilkS") (effects (font (size 1 1) (thickness 0.12))))
-    (pad "1" smd rect (at -28 0) (size 1.6 4) (layers "F.Cu" "F.Paste" "F.Mask") (net 1 "SOLAR_P"))
-    (pad "2" smd rect (at 28 0) (size 1.6 4) (layers "F.Cu" "F.Paste" "F.Mask") (net 3 "SOLAR_MID1"))
+    (pad "1" smd rect (at -27 0) (size 1.6 4) (layers "F.Cu" "F.Paste" "F.Mask") (net 1 "SOLAR_P"))
+    (pad "2" smd rect (at 27 0) (size 1.6 4) (layers "F.Cu" "F.Paste" "F.Mask") (net 3 "SOLAR_MID1"))
+    (fp_rect (start -28.05 -2.25) (end 28.05 2.25) (stroke (width 0.05) (type solid)) (fill no) (layer "F.CrtYd"))
     (model "${KIPRJMOD}/../3dmodels/cells/solar_cell_small_52.07x19.65x0.21.wrl"
       (offset
@@
     (fp_text user "+" (at -26 23.6) (layer "F.SilkS") (effects (font (size 1 1) (thickness 0.12))))
     (fp_text user "-" (at 26 23.6) (layer "F.SilkS") (effects (font (size 1 1) (thickness 0.12))))
-    (pad "1" smd rect (at -28 0) (size 1.6 4) (layers "F.Cu" "F.Paste" "F.Mask") (net 3 "SOLAR_MID1"))
-    (pad "2" smd rect (at 28 0) (size 1.6 4) (layers "F.Cu" "F.Paste" "F.Mask") (net 4 "SOLAR_MID2"))
+    (pad "1" smd rect (at -27 0) (size 1.6 4) (layers "F.Cu" "F.Paste" "F.Mask") (net 3 "SOLAR_MID1"))
+    (pad "2" smd rect (at 27 0) (size 1.6 4) (layers "F.Cu" "F.Paste" "F.Mask") (net 4 "SOLAR_MID2"))
+    (fp_rect (start -28.05 -2.25) (end 28.05 2.25) (stroke (width 0.05) (type solid)) (fill no) (layer "F.CrtYd"))
     (model "${KIPRJMOD}/../3dmodels/cells/solar_cell_small_52.07x19.65x0.21.wrl"
       (offset
@@
     (fp_text user "+" (at -26 23.6) (layer "F.SilkS") (effects (font (size 1 1) (thickness 0.12))))
     (fp_text user "-" (at 26 23.6) (layer "F.SilkS") (effects (font (size 1 1) (thickness 0.12))))
-    (pad "1" smd rect (at -28 0) (size 1.6 4) (layers "F.Cu" "F.Paste" "F.Mask") (net 4 "SOLAR_MID2"))
-    (pad "2" smd rect (at 28 0) (size 1.6 4) (layers "F.Cu" "F.Paste" "F.Mask") (net 2 "SOLAR_N"))
+    (pad "1" smd rect (at -27 0) (size 1.6 4) (layers "F.Cu" "F.Paste" "F.Mask") (net 4 "SOLAR_MID2"))
+    (pad "2" smd rect (at 27 0) (size 1.6 4) (layers "F.Cu" "F.Paste" "F.Mask") (net 2 "SOLAR_N"))
+    (fp_rect (start -28.05 -2.25) (end 28.05 2.25) (stroke (width 0.05) (type solid)) (fill no) (layer "F.CrtYd"))
+    (model "${KIPRJMOD}/../3dmodels/cells/solar_cell_small_52.07x19.65x0.21.wrl"
+      (offset
+        (xyz 0 0 0)
+      )
+      (scale
+        (xyz 1 1 1)
+      )
+      (rotate
+        (xyz 0 0 0)
+      )
+    )
+  )
+  (footprint "WingV9:SolarCell_52x19mm"
+    (layer "B.Cu")
+    (at 30 12.5)
+    (property "Reference" "SC4"
+      (at 0 0 0)
+      (layer "F.SilkS")
+      (hide yes)
+      (effects
+        (font
+          (size 1 1)
+          (thickness 0.15)
+        )
+      )
+    )
+    (property "Value" "SolarCell_52x19mm_0.5V"
+      (at 0 0 0)
+      (layer "F.Fab")
+      (hide yes)
+      (effects
+        (font
+          (size 1 1)
+          (thickness 0.15)
+        )
+      )
+    )
+    (attr smd)
+    (fp_rect (start -26 3) (end 26 22) (stroke (width 0.12) (type solid)) (fill no) (layer "B.SilkS"))
+    (fp_text user "+" (at 26 23.6) (layer "B.SilkS") (effects (font (size 1 1) (thickness 0.12))))
+    (fp_text user "-" (at -26 23.6) (layer "B.SilkS") (effects (font (size 1 1) (thickness 0.12))))
+    (pad "1" smd rect (at 27 0) (size 1.6 4) (layers "B.Cu" "B.Paste" "B.Mask") (net 1 "SOLAR_P"))
+    (pad "2" smd rect (at -27 0) (size 1.6 4) (layers "B.Cu" "B.Paste" "B.Mask") (net 3 "SOLAR_MID1"))
+    (fp_rect (start -28.05 -2.25) (end 28.05 2.25) (stroke (width 0.05) (type solid)) (fill no) (layer "B.CrtYd"))
+    (model "${KIPRJMOD}/../3dmodels/cells/solar_cell_small_52.07x19.65x0.21.wrl"
+      (offset
+        (xyz 0 0 0)
+      )
+      (scale
+        (xyz 1 1 1)
+      )
+      (rotate
+        (xyz 0 0 0)
+      )
+    )
+  )
+  (footprint "WingV9:SolarCell_52x19mm"
+    (layer "B.Cu")
+    (at 88 12.5)
+    (property "Reference" "SC5"
+      (at 0 0 0)
+      (layer "F.SilkS")
+      (hide yes)
+      (effects
+        (font
+          (size 1 1)
+          (thickness 0.15)
+        )
+      )
+    )
+    (property "Value" "SolarCell_52x19mm_0.5V"
+      (at 0 0 0)
+      (layer "F.Fab")
+      (hide yes)
+      (effects
+        (font
+          (size 1 1)
+          (thickness 0.15)
+        )
+      )
+    )
+    (attr smd)
+    (fp_rect (start -26 3) (end 26 22) (stroke (width 0.12) (type solid)) (fill no) (layer "B.SilkS"))
+    (fp_text user "+" (at 26 23.6) (layer "B.SilkS") (effects (font (size 1 1) (thickness 0.12))))
+    (fp_text user "-" (at -26 23.6) (layer "B.SilkS") (effects (font (size 1 1) (thickness 0.12))))
+    (pad "1" smd rect (at 27 0) (size 1.6 4) (layers "B.Cu" "B.Paste" "B.Mask") (net 3 "SOLAR_MID1"))
+    (pad "2" smd rect (at -27 0) (size 1.6 4) (layers "B.Cu" "B.Paste" "B.Mask") (net 4 "SOLAR_MID2"))
+    (fp_rect (start -28.05 -2.25) (end 28.05 2.25) (stroke (width 0.05) (type solid)) (fill no) (layer "B.CrtYd"))
+    (model "${KIPRJMOD}/../3dmodels/cells/solar_cell_small_52.07x19.65x0.21.wrl"
+      (offset
+        (xyz 0 0 0)
+      )
+      (scale
+        (xyz 1 1 1)
+      )
+      (rotate
+        (xyz 0 0 0)
+      )
+    )
+  )
+  (footprint "WingV9:SolarCell_52x19mm"
+    (layer "B.Cu")
+    (at 146 12.5)
+    (property "Reference" "SC6"
+      (at 0 0 0)
+      (layer "F.SilkS")
+      (hide yes)
+      (effects
+        (font
+          (size 1 1)
+          (thickness 0.15)
+        )
+      )
+    )
+    (property "Value" "SolarCell_52x19mm_0.5V"
+      (at 0 0 0)
+      (layer "F.Fab")
+      (hide yes)
+      (effects
+        (font
+          (size 1 1)
+          (thickness 0.15)
+        )
+      )
+    )
+    (attr smd)
+    (fp_rect (start -26 3) (end 26 22) (stroke (width 0.12) (type solid)) (fill no) (layer "B.SilkS"))
+    (fp_text user "+" (at 26 23.6) (layer "B.SilkS") (effects (font (size 1 1) (thickness 0.12))))
+    (fp_text user "-" (at -26 23.6) (layer "B.SilkS") (effects (font (size 1 1) (thickness 0.12))))
+    (pad "1" smd rect (at 27 0) (size 1.6 4) (layers "B.Cu" "B.Paste" "B.Mask") (net 4 "SOLAR_MID2"))
+    (pad "2" smd rect (at -27 0) (size 1.6 4) (layers "B.Cu" "B.Paste" "B.Mask") (net 2 "SOLAR_N"))
+    (fp_rect (start -28.05 -2.25) (end 28.05 2.25) (stroke (width 0.05) (type solid)) (fill no) (layer "B.CrtYd"))
     (model "${KIPRJMOD}/../3dmodels/cells/solar_cell_small_52.07x19.65x0.21.wrl"
       (offset
@@
     (fp_text user "N" (at -5 16.9) (layer "F.SilkS") (effects (font (size 0.6 0.6) (thickness 0.1))))
     (fp_rect (start -7 8.4) (end -3 16.6) (stroke (width 0.1) (type solid)) (fill none) (layer "F.SilkS"))
+    (fp_rect (start -7.25 8.95) (end -2.75 16.05) (stroke (width 0.05) (type solid)) (fill no) (layer "F.CrtYd"))
     (model "${KIPRJMOD}/../3dmodels/wing/wing_v9_tab_4pin_lands.wrl"
       (offset
@@
     )
     (pad "" np_thru_hole circle (at 0 0) (size 2.2 2.2) (drill 2.2) (layers "*.Cu" "*.Mask"))
+    (fp_circle (center 0 0) (end 1.35 0) (stroke (width 0.05) (type solid)) (fill no) (layer "F.CrtYd"))
   )
   (footprint "WingV9:MountingHole_2.2mm_NPTH"
@@
     )
     (pad "" np_thru_hole circle (at 0 0) (size 2.2 2.2) (drill 2.2) (layers "*.Cu" "*.Mask"))
+    (fp_circle (center 0 0) (end 1.35 0) (stroke (width 0.05) (type solid)) (fill no) (layer "F.CrtYd"))
   )
   (footprint "WingV9:MountingHole_2.2mm_NPTH"
@@
     )
     (pad "" np_thru_hole circle (at 0 0) (size 2.2 2.2) (drill 2.2) (layers "*.Cu" "*.Mask"))
+    (fp_circle (center 0 0) (end 1.35 0) (stroke (width 0.05) (type solid)) (fill no) (layer "F.CrtYd"))
   )
   (footprint "WingV9:Fiducial_1mm_Mask2mm"
@@
     (attr smd)
     (pad "1" smd circle (at 0 0) (size 1 1) (layers "F.Cu" "F.Mask"))
+    (fp_circle (center 0 0) (end 1.25 0) (stroke (width 0.05) (type solid)) (fill no) (layer "F.CrtYd"))
     (model "${KIPRJMOD}/../3dmodels/wing/wing_v9_fiducial_1mm_dot.wrl"
       (offset
@@
     (attr smd)
     (pad "1" smd circle (at 0 0) (size 1 1) (layers "F.Cu" "F.Mask"))
+    (fp_circle (center 0 0) (end 1.25 0) (stroke (width 0.05) (type solid)) (fill no) (layer "F.CrtYd"))
     (model "${KIPRJMOD}/../3dmodels/wing/wing_v9_fiducial_1mm_dot.wrl"
       (offset
@@
     (attr smd)
     (pad "1" smd circle (at 0 0) (size 1 1) (layers "F.Cu" "F.Mask"))
+    (fp_circle (center 0 0) (end 1.25 0) (stroke (width 0.05) (type solid)) (fill no) (layer "F.CrtYd"))
     (model "${KIPRJMOD}/../3dmodels/wing/wing_v9_fiducial_1mm_dot.wrl"
       (offset
@@
     (pad "1" smd rect (at -0.45 0) (size 0.5 0.6) (layers "F.Cu" "F.Paste" "F.Mask"))
     (pad "2" smd rect (at 0.45 0) (size 0.5 0.6) (layers "F.Cu" "F.Paste" "F.Mask"))
+    (fp_rect (start -0.95 -0.55) (end 0.95 0.55) (stroke (width 0.05) (type solid)) (fill no) (layer "F.CrtYd"))
     (model "${KIPRJMOD}/../3dmodels/wing/ferrite_bead_0402_dnp.wrl"
       (offset
@@
     (attr smd)
     (pad "1" smd rect (at 0 0) (size 2 2) (layers "F.Cu" "F.Mask"))
+    (fp_rect (start -1.25 -1.25) (end 1.25 1.25) (stroke (width 0.05) (type solid)) (fill no) (layer "F.CrtYd"))
     (model "${KIPRJMOD}/../3dmodels/wing/wing_v9_rf_provision_pad_2x2.wrl"
       (offset
